File: Hardware/Beefy_3.brd (EAGLE design)
At the start: 22.9 x 17.3 mm, 20 parts, among them U1 3.3V, U2 FTS31XS-U

Commit message: Added shield pour
Parts:
- moved C4 2.80 mm to (16.9, 2.26), turned to 0 degrees
Connections:
- new net SHIELD: JP1.SHIELD1, JP1.SHIELD2, JP1.SHIELD3
Routing:
- added copper zone on layer 1, net SHIELD
Changed lines of the file:
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@@
 <setting verticaltext="up"/>
 </settings>
-<grid distance="0.0008" unitdist="inch" unit="inch" style="lines" multiple="1" display="yes" altdistance="0.0001" altunitdist="inch" altunit="inch"/>
+<grid distance="0.01" unitdist="inch" unit="inch" style="lines" multiple="1" display="yes" altdistance="0.0001" altunitdist="inch" altunit="inch"/>
 <layers>
 <layer number="1" name="Top" color="4" fill="1" visible="yes" active="yes"/>
@@
 <layer number="199" name="Contour" color="7" fill="1" visible="no" active="yes"/>
 <layer number="200" name="200bmp" color="1" fill="10" visible="no" active="yes"/>
-<layer number="201" name="201bmp" color="2" fill="10" visible="yes" active="yes"/>
+<layer number="201" name="201bmp" color="2" fill="10" visible="no" active="yes"/>
 <layer number="202" name="202bmp" color="3" fill="1" visible="no" active="no"/>
 <layer number="203" name="203bmp" color="4" fill="10" visible="no" active="yes"/>
@@
 </class>
 </classes>
-<designrules name="SparkFun-2-layer *">
-<description language="en">&lt;b&gt;EAGLE Design Rules&lt;/b&gt;
+<designrules name="SparkFun-2-layer-TIGHT">
+<description language="en">&lt;b&gt;SparkFun 2 Layer Design Rule Checks - STANDARD/TIGHT/FAB-LIMIT&lt;/b&gt;
 &lt;p&gt;
-The default Design Rules have been set to cover
-a wide range of applications. Your particular design
-may have different requirements, so please make the
-necessary adjustments and save your customized
-design rules under a new name.</description>
+These rules have been curated by SparkFuns DFM commitee. After doing much research, communicating with our multiple fab houses, and getting quotes of various designs, we have compiled three DRU files.
+&lt;p&gt;
+&lt;b&gt;STANDARD:&lt;/b&gt; This is more of a &quot;best case scenario&quot; set of limitations. If your design has the space, and/or you have the time to work within these parameters, please do. Larger trace width and clearance makes for easier visual inspection of the PCB while troubleshooting (useful in production and to the end user). It also allows for better ability to hack a trace (if you are crazy enough to scrape away the mask and solder to a trace). Another thing to keep in mind is that more metal is just more robust.
+&lt;p&gt;
+&lt;b&gt;TIGHT:&lt;/b&gt; This is where cost comes into play. We have found that most fab houses begin to add extra charges when you go smaller than these specs. In some cases, going to less than 15 mil trace can increase the cost by 10%. (This is why we have set the min drill on this DRU to 15 mil) Same story for traces thinner than 7 mil. To avoid those extra charges, then stay within the rules of this DRU.
+&lt;p&gt;
+&lt;b&gt;FAB-LIMIT:&lt;/b&gt; These set of rules are at the very limit of most fab houses capabilities. You will pay more for these specs, and it should be used on designs that have a darned good reason to need 4 mil vias and 4 mil traces.
+&lt;p&gt;
+**NOTE Clearance, Distance, Sizes, and Restring are all set to different limits in each of these three DRU files. Please compare the files within the CAM job editor window of eagle to see all the numbers.
+&lt;p&gt;
+***NOTE, Please set your Net Classes to default (0mil for all settings), so that it won't effect the DRC when you run it with these settings.</description>
 <param name="layerSetup" value="(1*16)"/>
 <param name="mtCopper" value="0.035mm 0.035mm 0.035mm 0.035mm 0.035mm 0.035mm 0.035mm 0.035mm 0.035mm 0.035mm 0.035mm 0.035mm 0.035mm 0.035mm 0.035mm 0.035mm"/>
@@
 <param name="mdViaViaSameLayer" value="8mil"/>
 <param name="mnLayersViaInSmd" value="2"/>
-<param name="mdCopperDimension" value="8mil"/>
-<param name="mdDrill" value="8mil"/>
+<param name="mdCopperDimension" value="7mil"/>
+<param name="mdDrill" value="7mil"/>
 <param name="mdSmdStop" value="0mil"/>
 <param name="msWidth" value="7mil"/>
@@
 <param name="rvMicroViaOuter" value="0.25"/>
 <param name="rvMicroViaInner" value="0.25"/>
-<param name="rlMinPadTop" value="12mil"/>
+<param name="rlMinPadTop" value="7mil"/>
 <param name="rlMaxPadTop" value="20mil"/>
-<param name="rlMinPadInner" value="10mil"/>
+<param name="rlMinPadInner" value="7mil"/>
 <param name="rlMaxPadInner" value="20mil"/>
-<param name="rlMinPadBottom" value="12mil"/>
+<param name="rlMinPadBottom" value="7mil"/>
 <param name="rlMaxPadBottom" value="20mil"/>
-<param name="rlMinViaOuter" value="10mil"/>
+<param name="rlMinViaOuter" value="7mil"/>
 <param name="rlMaxViaOuter" value="20mil"/>
-<param name="rlMinViaInner" value="10mil"/>
+<param name="rlMinViaInner" value="7mil"/>
 <param name="rlMaxViaInner" value="20mil"/>
 <param name="rlMinMicroViaOuter" value="4mil"/>
@@
 <attribute name="PROD_ID" value="CAP-00810" x="12.065" y="13.5382" size="1.778" layer="27" rot="R90" display="off"/>
 </element>
-<element name="C4" library="SparkFun-Capacitors" package="EIA3216" value="10uF" x="19.7104" y="2.2098" smashed="yes" rot="R180">
-<attribute name="NAME" x="22.2504" y="0.8288" size="0.4064" layer="25" rot="R180"/>
-<attribute name="VALUE" value="10uF" x="22.5664" y="2.8178" size="0.4064" layer="27" rot="R270"/>
-<attribute name="PROD_ID" value="CAP-00811" x="19.7104" y="2.2098" size="1.778" layer="27" rot="R180" display="off"/>
+<element name="C4" library="SparkFun-Capacitors" package="EIA3216" value="10uF" x="16.906240625" y="2.2606" smashed="yes">
+<attribute name="NAME" x="14.366240625" y="3.6416" size="0.4064" layer="25"/>
+<attribute name="VALUE" value="10uF" x="14.050240625" y="1.6526" size="0.4064" layer="27" rot="R90"/>
+<attribute name="PROD_ID" value="CAP-00811" x="16.906240625" y="2.2606" size="1.778" layer="27" display="off"/>
 </element>
 <element name="C5" library="SparkFun-Capacitors" package="0603-CAP" value="0.1uF" x="13.3096" y="13.5382" smashed="yes" rot="R90">
@@
 <via x="19.1262" y="5.3086" extent="1-16" drill="0.381"/>
 <via x="18.1102" y="5.3086" extent="1-16" drill="0.381"/>
-<wire x1="18.3104" y1="2.2098" x2="18.3104" y2="5.3086" width="1.016" layer="1"/>
-<wire x1="18.3104" y1="5.3086" x2="18.1102" y2="5.3086" width="1.016" layer="1"/>
+<wire x1="18.306240625" y1="5.3086" x2="18.1102" y2="5.3086" width="1.016" layer="1"/>
 <wire x1="17.0942" y1="5.3086" x2="17.0942" y2="6.9342" width="0.6604" layer="16"/>
 <wire x1="17.0942" y1="6.9342" x2="15.9512" y2="8.0772" width="0.6604" layer="16"/>
@@
 <wire x1="11.7475" y1="9.9187" x2="10.4648" y2="8.636" width="0.254" layer="1"/>
 <wire x1="10.4648" y1="8.636" x2="9.3218" y2="8.636" width="0.254" layer="1"/>
+<wire x1="18.3104" y1="5.3086" x2="18.306240625" y2="5.3086" width="1.016" layer="1"/>
+<wire x1="18.306240625" y1="5.3086" x2="18.306240625" y2="2.2606" width="1.016" layer="1"/>
 </signal>
 <signal name="3V3" class="1">
@@
 <wire x1="9.525" y1="2.286" x2="11.426" y2="2.286" width="0.254" layer="16"/>
 </signal>
-<signal name="N$3">
+<signal name="SHIELD">
+<polygon width="0.6096" layer="1" rank="2">
+<vertex x="22.86" y="13.97"/>
+<vertex x="19.304" y="13.97"/>
+<vertex x="19.304" y="3.302"/>
+<vertex x="22.86" y="3.302"/>
+</polygon>
 <via x="20.767040625" y="11.927840625" extent="1-16" drill="0.381"/>
-</signal>
-<signal name="N$4">
+<via x="20.685759375" y="5.36448125" extent="1-16" drill="0.381"/>
 <via x="20.84831875" y="8.81888125" extent="1-16" drill="0.381"/>
-</signal>
-<signal name="N$5">
-<via x="20.685759375" y="5.36448125" extent="1-16" drill="0.381"/>
+<contactref element="JP1" pad="SHIELD3"/>
+<contactref element="JP1" pad="SHIELD1"/>
+<contactref element="JP1" pad="SHIELD2"/>
 </signal>
 </signals>

Commit message: Added flame logo to top and clarified schematic note
Parts:
- added LOGO3: SFE_LOGO_FLAME.1_INCH, SparkFun-Aesthetics:SFE_LOGO_FLAME_.1
Changed lines of the file:
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@@
 <attribute name="PROD_ID" value="CONN-11752" x="20.8534" y="8.636" size="1.778" layer="27" rot="R180" display="off"/>
 </element>
+<element name="LOGO3" library="SparkFun-Aesthetics" package="SFE_LOGO_FLAME_.1" value="SFE_LOGO_FLAME.1_INCH" x="17.272" y="12.7" rot="R90"/>
 </elements>
 <signals>

Commit message: moved board fids
Parts:
- moved JP4 17.8 mm to (18.7, 2.18)
- moved JP6 7.38 mm to (14.6, 15.8)
- moved JP5 3.09 mm to (18.9, 15.8)
- moved JP3 1.27 mm to (4.09, 1.68)
