File: Production/Beefy_3_Panel_v10.brd (EAGLE design)
At the start: 226.6 x 119.9 mm, 963 parts, among them U1 3.3V, U10 FTS31XS-U, U11 3.3V, U12 FTS31XS-U, U13 3.3V, U14 FTS31XS-U, U15 3.3V, U16 FTS31XS-U, U17 3.3V, U18 FTS31XS-U, U19 3.3V, U2 FTS31XS-U, U20 FTS31XS-U, U21 3.3V, U22 FTS31XS-U, U23 3.3V, U24 FTS31XS-U, U25 3.3V, U26 FTS31XS-U, U27 3.3V, U28 FTS31XS-U, U29 3.3V, U3 3.3V, U30 FTS31XS-U, U31 3.3V, U32 FTS31XS-U, U33 3.3V, U34 FTS31XS-U, U35 3.3V, U36 FTS31XS-U, U37 3.3V, U38 FTS31XS-U, U39 3.3V, U4 FTS31XS-U, U40 FTS31XS-U, U41 3.3V, U42 FTS31XS-U, U43 3.3V, U44 FTS31XS-U, U45 3.3V, U46 FTS31XS-U, U47 3.3V, U48 FTS31XS-U, U49 3.3V, U5 3.3V, U50 FTS31XS-U, U51 3.3V, U52 FTS31XS-U, U53 3.3V, U54 FTS31XS-U, U55 3.3V, U56 FTS31XS-U, U57 3.3V, U58 FTS31XS-U, U59 3.3V, U6 FTS31XS-U, U60 FTS31XS-U, U61 3.3V, U62 FTS31XS-U, U63 3.3V, U64 FTS31XS-U, U65 3.3V, U66 FTS31XS-U, U67 3.3V, U68 FTS31XS-U, U69 3.3V, U7 3.3V, U70 FTS31XS-U, U71 3.3V, U72 FTS31XS-U, U73 3.3V, U74 FTS31XS-U, U75 3.3V, U76 FTS31XS-U, U77 3.3V, U78 FTS31XS-U, U79 3.3V, U8 FTS31XS-U, U80 FTS31XS-U, U81 3.3V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

Commit message: added bottom side panel fiducials
Parts:
- added E$2: (no value), SparkFun-Retired:FIDUCIAL-1.5X3
- added E$3, E$4: (no value), SparkFun-Aesthetics:FIDUCIAL-1X2
Changed lines of the file:
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@@
 <element name="E$8" library="SparkFun-Aesthetics" package="FIDUCIAL-1X2" value="" x="11.43" y="114.681" rot="R270"/>
 <element name="E$1" library="SparkFun-Retired" package="FIDUCIAL-1.5X3" value="" x="11.938" y="4.572"/>
+<element name="E$2" library="SparkFun-Retired" package="FIDUCIAL-1.5X3" value="" x="11.938" y="4.572" rot="MR0"/>
+<element name="E$3" library="SparkFun-Aesthetics" package="FIDUCIAL-1X2" value="" x="11.43" y="114.681" rot="MR270"/>
+<element name="E$4" library="SparkFun-Aesthetics" package="FIDUCIAL-1X2" value="" x="207.772" y="114.681" rot="MR90"/>
 </elements>
 <signals>
